File: hardware/ZSWatch-Dock.kicad_pcb (KiCad board)
At the start: 4 copper layers, 80 x 48 mm, 71 parts, among them IC101 TLV70218_SOT23-5, IC102 FT230XQ, IC103 MIC5219-3.3YM5, IC104 NTS0104GU12, IC105 USBLC6-2P6, IC106 USB2512BT, IC107 USBLC6-2P6, IC108 MIC2026-1xM, J102 Voltage, Q101 BSH205G2AR, SW101 Reset, SW102 Charge, X101 Debug, X102 UART, X103 Host, X104 Device, X105 Current, Y101 24 MHz

Commit message: Dock: Revision 1
- Fix wrong title for USB Host and Device
- Fix missing VBus for +3V3 and +1V8 rail

- Set revision to 1

Signed-off-by: Daniel Kampert <danielkampert@kampis-elektroecke.de>
Parts:
- IC104: value NTS0104GU12 -> NTS0104PW,118
Connections:
- IC101 pad 1: V_{Watch} -> V_{BUS}
- IC101 pad 3: V_{Watch} -> V_{BUS}
- IC103 pad 1: V_{Watch} -> V_{BUS}
- IC103 pad 3: V_{Watch} -> V_{BUS}
Routing:
- net V_{BUS}: track 33.9 -> 74.7 mm
- net V_{Watch}: track 153.0 -> 143.5 mm, vias 5 -> 3

Commit message: Bug: Issue #45
Signed-off-by: Daniel Kampert <DanielKampert@kampis-elektroecke.de>
Parts:
- removed the SW101 at (141.1, 137.8)
- added S101: Reset, Wuerth:WS-TASV-6x6, F.Cu at (141.1, 137.8)
- renumbered R110 to R109, R109 to R110, SW102 to SW101
Routing:
- net GND: track 62.5 -> 59.7 mm, vias 46 -> 45
- net RESETn: track 55.8 -> 53.8 mm

Commit message: Issue #46
Parts:
- IC104: value NTS0104PW,118 -> NL3V4T244MU2TAG-Q
Changed lines of the file:
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@@
 			)
 		)
-		(property "Value" "NTS0104PW,118"
+		(property "Value" "NL3V4T244MU2TAG-Q"
 			(at 0 3.45 0)
 			(layer "F.Fab")
@@
 			)
 		)
-		(property "Datasheet" "https://www.onsemi.com/download/data-sheet/pdf/nl3v4t244-d.pdf"
+		(property "Datasheet" "https://www.mouser.de/datasheet/2/308/1/NL3V4T244_D-3579604.pdf"
 			(at 0 0 0)
 			(layer "F.Fab")
@@
 			)
 		)
-		(property "manf" "NXP Semiconductors"
+		(property "manf" "onsemi"
 			(at 0 0 0)
 			(unlocked yes)
@@
 			)
 		)
-		(property "manf#" "NTS0104PW,118"
+		(property "manf#" "NL3V4T244MU2TAG-Q"
 			(at 0 0 0)
 			(unlocked yes)
@@
 			)
 		)
-		(property "mouser#" "771-NTS0104PW118"
+		(property "mouser#" "863-NL3V4T244MU2TAG-Q"
 			(at 0 0 0)
 			(unlocked yes)

Commit message: Issue #47, Issue #48
Parts:
- added R103: 0R, Resistor_SMD:R_0805_2012Metric, F.Cu at (148.4, 97.1)
- added R104: 0R, Resistor_SMD:R_0805_2012Metric, F.Cu at (151.8, 97.1)
- renumbered R103 to R105, R104 to R106, R105 to R107, R106 to R108, R107 to R109, R108 to R110, R109 to R111, R110 to R112, R111 to R113, R112 to R114, R113 to R115, R114 to R116, R115 to R117, R116 to R118, R117 to R119
Connections:
- IC104 pad 14: +1V8 -> Net-(IC104-OE)
- X104 pad A10: SWDIO_{LV} -> TxD_{LV}
- X104 pad A11: SWDCLK_{LV} -> RxD_{LV}
- X104 pad A2: RxD_{LV} -> SWDCLK_{LV}
- X104 pad A3: TxD_{LV} -> SWDIO_{LV}
- X104 pad B10: SWDIO_{LV} -> TxD_{LV}
- X104 pad B11: SWDCLK_{LV} -> RxD_{LV}
- X104 pad B2: RxD_{LV} -> SWDCLK_{LV}
- X104 pad B3: TxD_{LV} -> SWDIO_{LV}
Routing:
- net SWDIO_{LV}: track 39.8 -> 27.4 mm
- net SWDCLK_{LV}: track 38.0 -> 26.1 mm
- net TxD_{LV}: track 72.5 -> 84.4 mm
- net RxD_{LV}: track 94.5 -> 105.5 mm, vias 5 -> 6
- net Net-(IC104-OE): track 0.00 -> 4.88 mm
- net +1V8: track 77.5 -> 75.3 mm
- net GND: track 59.7 -> 60.2 mm, vias 45 -> 46

Commit message: Feature: Issue #54 and Issue #50
Signed-off-by: Daniel Kampert <DanielKampert@kampis-elektroecke.de>
Parts:
- removed the D103 at (157.8, 102.3)
- removed the D104 at (156.3, 102.3)
- removed D105, D106: ESD5Zxx, Diode_SMD:D_SOD-523
- added IC102: USBLC6-2P6, Package_TO_SOT_SMD:SOT-666, F.Cu at (155.7, 102.6)
- added SB101: Resetn, Jumper:SolderJumper-2_P1.3mm_Open_RoundedPad1.0x1.5mm, B.Cu at (149.7, 97.9)
- added SB102: SWDCLK, Jumper:SolderJumper-2_P1.3mm_Open_RoundedPad1.0x1.5mm, B.Cu at (149.7, 100.5)
- added SB103: SWDIO, Jumper:SolderJumper-2_P1.3mm_Open_RoundedPad1.0x1.5mm, B.Cu at (149.6, 102.5)
- R107: value 1k -> 3k3
- moved D101 2.12 mm to (158.3, 98.9)
- moved D102 2.12 mm to (159.8, 98.9)
- moved C109 0.34 mm to (147.7, 104.4)
- renumbered D107 to D103, D108 to D104, IC102 to IC103, IC103 to IC104, IC104 to IC105, IC105 to IC106, IC106 to IC107, IC107 to IC108, IC108 to IC109
Connections:
- IC105 pad 10: Net-(D103-A) (its old number) -> Net-(IC105-B3)
- IC105 pad 8: Net-(D105-A) -> Net-(IC105-B4)
- X101 pad 2: Net-(D105-A) -> Net-(X101-SWDIO/TMS)
- X101 pad 4: Net-(D103-A) (its old number) -> Net-(X101-SWCLK/TCK)
Routing:
- net Net-(D105-A): track 17.6 -> 0.00 mm
- net Net-(D101-K): track 47.3 -> 30.6 mm, vias 4 -> 2
- net Net-(D103-A) (its old number): track 15.7 -> 0.00 mm, vias 2 -> 0
- net Net-(X101-SWDIO/TMS): track 0.00 -> 13.1 mm
- net Net-(X101-SWCLK/TCK): track 0.00 -> 11.8 mm, vias 0 -> 2
- net RESETn_{LV}: track 32.7 -> 40.1 mm
- net Net-(IC105-B3): track 0.00 -> 5.60 mm, vias 0 -> 1
- net Net-(IC105-B4): track 0.00 -> 4.85 mm, vias 0 -> 1
- net SWDCLK_{LV}: track 26.1 -> 29.8 mm
- net RESETn: track 53.8 -> 56.7 mm, vias 2 -> 3
- net SWDIO_{LV}: track 27.4 -> 30.0 mm, vias 5 -> 6
- net Net-(D101-A): track 10.9 -> 13.3 mm
- net GND: track 60.2 -> 59.5 mm, vias 46 -> 45

Commit message: Feature: Issue #52
Signed-off-by: Daniel Kampert <DanielKampert@kampis-elektroecke.de>
Parts:
- added R120: 22R, Resistor_SMD:R_0603_1608Metric, F.Cu at (158.8, 103.6)
- added R121: 22R, Resistor_SMD:R_0603_1608Metric, F.Cu at (158.8, 102.0)
- moved SB103 0.51 mm to (149.7, 103.0)
- moved C109 0.20 mm to (147.9, 104.4)
Connections:
- D101 pad 2: Net-(D101-A) -> RESETn
- D102 pad 1: Net-(D101-A) -> RESETn
- IC102 pad 4: Net-(X101-SWDIO/TMS) -> Net-(IC102-I/O2-Pad4)
- IC102 pad 6: Net-(X101-SWCLK/TCK) -> Net-(IC102-I/O1-Pad6)
- IC105 pad 11: Net-(D101-A) -> RESETn
- X101 pad 10: Net-(D101-A) -> RESETn
Routing:
- net RESETn: track 56.7 -> 70.7 mm
- net Net-(D101-A): track 13.3 -> 0.00 mm
- net Net-(X101-SWDIO/TMS): track 13.1 -> 9.78 mm
- net Net-(X101-SWCLK/TCK): track 11.8 -> 8.73 mm
- net Net-(IC102-I/O2-Pad4): track 0.00 -> 1.91 mm
- net Net-(IC102-I/O1-Pad6): track 0.00 -> 1.42 mm
- net Net-(IC105-~{OE}): track 4.88 -> 4.05 mm
