File: hardware/ZSWatch-Dock.kicad_pcb (KiCad board)
At the start: 4 copper layers, 80 x 48 mm, 75 parts, among them IC101 TLV70218_SOT23-5, IC102 USBLC6-2P6, IC103 FT230XQ, IC104 MIC5219-3.3YM5, IC105 NL3V4T244MU2TAG-Q, IC106 USBLC6-2P6, IC107 USB2512BT, IC108 USBLC6-2P6, IC109 MIC2026-1xM, J102 Voltage, Q101 BSH205G2AR, SW101 Charge, X101 Debug, X102 UART, X103 Host, X104 Device, X105 Current, Y101 24 MHz

Commit message: Issue #51, Clean up Copy+Paste errors in Schematics
Connections:
- IC108 pad 5: Net-(IC108-VBUS) -> V_{Watch}
- Q101 pad 1: Net-(Q101-G) -> Net-(D104-K)
- R115 pad 2: Net-(IC108-VBUS) -> Net-(X105-Pin_1)
- R117 pad 1: Net-(Q101-G) -> Net-(D104-K)
- SW101 pad 1: Net-(D104-K) -> unconnected-(SW101A-A-Pad1)
- SW101 pad 3: Net-(Q101-G) -> Net-(D104-K)
- X104 pad A4: Net-(IC108-VBUS) -> Net-(X105-Pin_1)
- X104 pad A9: Net-(IC108-VBUS) -> Net-(X105-Pin_1)
- X104 pad B4: Net-(IC108-VBUS) -> Net-(X105-Pin_1)
- X104 pad B9: Net-(IC108-VBUS) -> Net-(X105-Pin_1)
- X105 pad 1: Net-(IC108-VBUS) -> Net-(X105-Pin_1)
Routing:
- net Net-(Q101-G): track 38.9 -> 0.00 mm, vias 2 -> 0
- net Net-(D104-K): track 12.1 -> 47.7 mm, vias 2 -> 3
- net Net-(IC108-VBUS): track 27.3 -> 0.00 mm, vias 5 -> 0
- net Net-(X105-Pin_1): track 0.00 -> 27.0 mm, vias 0 -> 2
- net V_{Watch}: track 143.5 -> 158.3 mm
