File: hardware/ZSWatch-Dock.kicad_pcb (KiCad board)
At the start: 4 copper layers, 80 x 48 mm, 75 parts, among them IC101 TLV70218_SOT23-5, IC102 USBLC6-2P6, IC103 FT230XQ, IC104 MIC5219-3.3YM5, IC105 NL3V4T244MU2TAG-Q, IC106 USBLC6-2P6, IC107 USB2512BT, IC108 USBLC6-2P6, IC109 MIC2026-1xM, J102 Voltage, Q101 BSH205G2AR, SW101 Charge, X101 Debug, X102 UART, X103 Host, X104 Device, X105 Current, Y101 24 MHz

Commit message: Feature: Issue #59
Signed-off-by: Daniel Kampert <DanielKampert@kampis-elektroecke.de>
Parts:
- removed IC105: NL3V4T244MU2TAG-Q, Package_SO:TSSOP-14_4.4x5mm_P0.65mm
- added IC405: TXB0304RUT, Package_DFN_QFN:Texas_R-PUQFN-N12, F.Cu at (192.3, 128.6)
- moved C409 5.39 mm to (189.6, 127.2)
- moved C406 2.06 mm to (195.0, 127.2), turned to 0 degrees
- moved SB403 0.20 mm to (192.4, 131.3)
- renumbered C101 to C401, C102 to C402, C103 to C403, C104 to C404, C105 to C405, C107 to C406, C106 to C407, C108 to C408, C109 to C409, C110 to C410, C111 to C411, C112 to C412, C113 to C413, C114 to C414, C115 to C415, C116 to C416, C117 to C417, C118 to C418, C119 to C419, D101 to D401, D102 to D402, D103 to D403, D104 to D404, IC101 to IC401, IC102 to IC402, IC103 to IC403, IC104 to IC404, IC106 to IC406, IC107 to IC407, IC108 to IC408, IC109 to IC409, J102 to J402, Q101 to Q401, R101 to R401, R121 to R402, R120 to R403, R102 to R404, R103 to R405, R104 to R406, R107 to R407, R108 to R408, R105 to R409, R106 to R410, R109 to R411, R110 to R412, R111 to R413, R112 to R414, R113 to R415, R114 to R416, R116 to R417, R115 to R418, R119 to R419, R117 to R420, R118 to R421, S101 to S401, SB101 to SB401, SB102 to SB402, SB103 to SB403, SW101 to SW401, X101 to X401, X102 to X402, X103 to X403, X104 to X404, X105 to X405, Y101 to Y401
Routing:
- net SWDIO_{LV}: track 30.3 -> 34.3 mm, vias 6 -> 5
- net Net-(IC405-B4): track 4.71 -> 7.29 mm
- net RESETn: track 70.7 -> 72.8 mm, vias 3 -> 4
- net RxD_{LV}: track 105.5 -> 103.5 mm
- net RESETn_{LV}: track 40.1 -> 42.0 mm
- net TxD_{LV}: track 84.4 -> 82.5 mm
- net Net-(IC405-B3): track 5.60 -> 6.66 mm
- net Net-(D401-K): track 30.6 -> 29.6 mm
- net GND: track 59.5 -> 58.8 mm, vias 45 -> 46
- net SWDCLK_{LV}: track 29.8 -> 29.5 mm, vias 3 -> 4
- net +1V8: track 75.0 -> 74.9 mm, vias 4 -> 5

Commit message: Issue #61
Parts:
- X404: footprint Connector_USB:USB_C_Receptacle_Amphenol_12401610E4-2A -> Amphenol:10133475-10001LF
- moved R416 14.1 mm to (177.0, 150.2), turned to 180 degrees
- moved R415 11.1 mm to (177.0, 146.5)
- moved X404 6.80 mm to (168.7, 148.3)
- moved IC408 6.53 mm to (177.0, 148.3)
Routing:
- net SWDCLK_{LV}: track 29.5 -> 44.7 mm
- net SWDIO_{LV}: track 34.3 -> 47.8 mm, vias 5 -> 3
- net /Project Architecture/Main/D_{2}+: track 3.81 -> 14.6 mm, vias 0 -> 2
- net RESETn_{LV}: track 42.0 -> 51.7 mm, vias 6 -> 5
- net /Project Architecture/Main/D_{2}-: track 4.96 -> 13.6 mm, vias 2 -> 1
- net V_{Watch}: track 158.3 -> 166.5 mm
- net RxD_{LV}: track 103.5 -> 95.5 mm, vias 6 -> 5
- net Net-(X405-Pin_1): track 27.0 -> 34.3 mm, vias 2 -> 3
- net TxD_{LV}: track 82.5 -> 75.8 mm, vias 3 -> 2
- net Net-(D404-K): track 47.7 -> 52.9 mm
- net USB-2-D-: track 45.2 -> 50.1 mm
- net USB-2-D+: track 45.9 -> 50.8 mm
- net Net-(X404-CC2): track 9.33 -> 10.6 mm, vias 0 -> 1
- net RESETn: track 72.8 -> 73.9 mm
- net Net-(X404-CC1): track 7.24 -> 7.97 mm
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Other:
- outline, holes or cut-outs redrawn
