File: hardware/ZSWatch-Dock.kicad_sch (KiCad schematic)
At the start: 63 parts, among them IC101 TLV70218_SOT23-5, IC102 FT230XQ, IC103 MIC5219-3.3YM5, IC104 NTS0104PW,118, IC105 USBLC6-2P6, IC106 USB2512BT, IC107 USBLC6-2P6, IC108 MIC2026-1xM, J101 Jumper, J102 Voltage, Q101 BSH205G2AR, SW101 Reset, SW102 Charge, X101 Debug, X102 UART, X103 Host, X104 Device, X105 Current, Y101 24 MHz

Commit message: Dock: Revision 1
- Fix wrong title for USB Host and Device
- Fix missing VBus for +3V3 and +1V8 rail

- Set revision to 1

Signed-off-by: Daniel Kampert <danielkampert@kampis-elektroecke.de>
Parts:
- R103, R104: now fitted
Connections:
- net V_{BUS}: now also IC101.1 (IN), IC101.3 (EN), IC103.1 (IN), IC103.3 (EN)
- net V_{Watch}: no longer IC101.1 (IN), IC101.3 (EN), IC103.1 (IN), IC103.3 (EN)
Changed lines of the file:
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@@
 	(title_block
 		(title "ZSWatch Dock v2")
-		(date "2025-05-24")
-		(rev "0")
+		(date "2025-07-11")
+		(rev "1")
 		(company "github.com/ZSWatch/Dock-HW")
 	)
@@
 		)
 	)
-	(text "USB (To Client/ZSWatch)"
+	(text "USB (To Host/Computer)"
 		(exclude_from_sim no)
 		(at 138.43 19.05 0)
@@
 		)
 	)
-	(text "USB (To Host/Computer)"
+	(text "USB (To Client/ZSWatch)"
 		(exclude_from_sim no)
 		(at 222.25 19.05 0)
@@
 		)
 	)
+	(global_label "V_{BUS}"
+		(shape input)
+		(at 81.28 29.21 180)
+		(fields_autoplaced yes)
+		(effects
+			(font
+				(size 1.27 1.27)
+			)
+			(justify right)
+		)
+		(property "Intersheetrefs" "${INTERSHEET_REFS}"
+			(at 74.7616 29.21 0)
+			(effects
+				(font
+					(size 1.27 1.27)
+				)
+				(justify right)
+				(hide yes)
+			)
+		)
+	)
 	(global_label "RESETn"
 		(shape output)
@@
 		)
 	)
-	(global_label "USB-1-D+"
-		(shape bidirectional)
-		(at 321.31 179.07 0)
+	(global_label "V_{BUS}"
+		(shape input)
+		(at 24.13 29.21 180)
 		(fields_autoplaced yes)
 		(effects
@@
 				(size 1.27 1.27)
 			)
-			(justify left)
+			(justify right)
 		)
 		(property "Intersheetrefs" "${INTERSHEET_REFS}"
-			(at 335.6002 179.07 0)
+			(at 17.6116 29.21 0)
 			(effects
 				(font
 					(size 1.27 1.27)
 				)
-				(justify left)
+				(justify right)
 				(hide yes)
 			)
 		)
 	)
-	(global_label "V_{Watch}"
-		(shape input)
-		(at 81.28 29.21 180)
+	(global_label "USB-1-D+"
+		(shape bidirectional)
+		(at 321.31 179.07 0)
 		(fields_autoplaced yes)
 		(effects
@@
 				(size 1.27 1.27)
 			)
-			(justify right)
+			(justify left)
 		)
 		(property "Intersheetrefs" "${INTERSHEET_REFS}"
-			(at 73.3586 29.21 0)
+			(at 335.6002 179.07 0)
 			(effects
 				(font
 					(size 1.27 1.27)
 				)
-				(justify right)
+				(justify left)
 				(hide yes)
 			)
@@
 		)
 	)
-	(global_label "V_{Watch}"
-		(shape input)
-		(at 24.13 29.21 180)
-		(fields_autoplaced yes)
-		(effects
-			(font
-				(size 1.27 1.27)
-			)
-			(justify right)
-		)
-		(property "Intersheetrefs" "${INTERSHEET_REFS}"
-			(at 16.2086 29.21 0)
-			(effects
-				(font
-					(size 1.27 1.27)
-				)
-				(justify right)
-				(hide yes)
-			)
-		)
-	)
 	(global_label "RxD_{LV}"
 		(shape output)
@@
 		(in_bom yes)
 		(on_board yes)
-		(dnp yes)
+		(dnp no)
 		(fields_autoplaced yes)
 		(property "Reference" "R104"
@@
 		(in_bom yes)
 		(on_board yes)
-		(dnp yes)
+		(dnp no)
 		(fields_autoplaced yes)
 		(property "Reference" "R103"

Commit message: Bug: Issue #44
Signed-off-by: Daniel Kampert <DanielKampert@kampis-elektroecke.de>
Parts:
- X101: manf# 623310235521 -> 62101021021; mouser# 710-623310235521 -> 710-62101021021
Changed lines of the file:
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@@
 			)
 		)
-		(property "Datasheet" "http://infocenter.arm.com/help/topic/com.arm.doc.ddi0314h/DDI0314H_coresight_components_trm.pdf"
+		(property "Datasheet" "https://www.we-online.com/components/products/datasheet/62101021021.pdf"
 			(at 25.4 124.46 90)
 			(effects
@@
 			)
 		)
-		(property "manf#" "623310235521"
+		(property "manf#" "62101021021"
 			(at 34.29 92.71 0)
 			(effects
@@
 			)
 		)
-		(property "mouser#" "710-623310235521"
+		(property "mouser#" "710-62101021021"
 			(at 34.29 92.71 0)
 			(effects

Commit message: Bug: Issue #45
Signed-off-by: Daniel Kampert <DanielKampert@kampis-elektroecke.de>
Parts:
- removed SW101: Reset, Wuerth:WS-TASV-6x6, symbol Switch:SW_MEC_5E
- added S101: Reset, Wuerth:WS-TASV-6x6, symbol Switch:SW_Push
- renumbered R110 to R109, R109 to R110, SW102 to SW101
Connections:
- net GND: now also S101.2
- net RESETn: now also S101.1

Commit message: Issue #46
Parts:
- IC104: value NTS0104PW,118 -> NL3V4T244MU2TAG-Q; manf NXP Semiconductors -> onsemi; manf# NTS0104PW,118 -> NL3V4T244MU2TAG-Q; mouser# 771-NTS0104PW118 -> 863-NL3V4T244MU2TAG-Q
Changed lines of the file:
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@@
 			)
 		)
-		(property "Value" "NTS0104PW,118"
+		(property "Value" "NL3V4T244MU2TAG-Q"
 			(at 95.25 96.52 0)
 			(effects
@@
 			)
 		)
-		(property "Datasheet" "https://www.onsemi.com/download/data-sheet/pdf/nl3v4t244-d.pdf"
+		(property "Datasheet" "https://www.mouser.de/datasheet/2/308/1/NL3V4T244_D-3579604.pdf"
 			(at 105.41 86.36 0)
 			(effects
@@
 			)
 		)
-		(property "manf" "NXP Semiconductors"
+		(property "manf" "onsemi"
 			(at 105.41 86.36 0)
 			(effects
@@
 			)
 		)
-		(property "manf#" "NTS0104PW,118"
+		(property "manf#" "NL3V4T244MU2TAG-Q"
 			(at 105.41 86.36 0)
 			(effects
@@
 			)
 		)
-		(property "mouser#" "771-NTS0104PW118"
+		(property "mouser#" "863-NL3V4T244MU2TAG-Q"
 			(at 105.41 86.36 0)
 			(effects

Commit message: Issue #47, Issue #48
Parts:
- added R103, R104: 0R, Resistor_SMD:R_0805_2012Metric, symbol Device:R_Small
- renumbered R103 to R105, R104 to R106, R105 to R107, R106 to R108, R107 to R109, R108 to R110, R109 to R111, R110 to R112, R111 to R113, R112 to R114, R113 to R115, R114 to R116, R115 to R117, R116 to R118, R117 to R119
Connections:
- net +1V8: now also R103.1; no longer IC104.14 (OE)
- net GND: now also R104.2
- net RxD_{LV}: now also X104.A11 (RX2+), X104.B11 (RX1+); no longer X104.A2 (TX1+), X104.B2 (TX2+)
- net SWDCLK_{LV}: now also X104.A2 (TX1+), X104.B2 (TX2+); no longer X104.A11 (RX2+), X104.B11 (RX1+)
- net SWDIO_{LV}: now also X104.A3 (TX1-), X104.B3 (TX2-); no longer X104.A10 (RX2-), X104.B10 (RX1-)
- net TxD_{LV}: now also X104.A10 (RX2-), X104.B10 (RX1-); no longer X104.A3 (TX1-), X104.B3 (TX2-)
- new net: IC104.14 (~{OE}), R103.2, R104.1

Commit message: Bug: Issue #49
Signed-off-by: Daniel Kampert <DanielKampert@kampis-elektroecke.de>
Parts:
- R107: value 1k -> 3k3; manf# CRCW06031K00FKEA -> CRCW06033K300FKEA; mouser# 71-CRCW06031K00FKEA -> 71-CRCW06033K300FKEA
Changed lines of the file:
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@@
 			)
 		)
-		(property "Value" "1k"
+		(property "Value" "3k3"
 			(at 186.69 190.5 90)
 			(effects
@@
 			)
 		)
-		(property "manf#" "CRCW06031K00FKEA"
+		(property "manf#" "CRCW06033K300FKEA"
 			(at 186.69 193.04 0)
 			(effects
@@
 			)
 		)
-		(property "mouser#" "71-CRCW06031K00FKEA"
+		(property "mouser#" "71-CRCW06033K300FKEA"
 			(at 186.69 193.04 0)
 			(effects
@@
 		(fields_autoplaced yes)
 		(property "Reference" "SW101"
-			(at 345.44 58.4199 90)
+			(at 346.71 58.4199 90)
 			(effects
 				(font
@@
 		)
 		(property "Value" "Charge"
-			(at 345.44 60.9599 90)
+			(at 346.71 60.9599 90)
 			(effects
 				(font
@@
 			)
 		)
-		(property "Datasheet" "~"
+		(property "Datasheet" "https://ckswitches.com/media/1424/pcm.pdf"
 			(at 341.63 59.69 0)
 			(effects

Commit message: Feature: Issue #54 and Issue #50
Signed-off-by: Daniel Kampert <DanielKampert@kampis-elektroecke.de>
Parts:
- removed D103, D104, D105, D106: ESD5Zxx, Diode_SMD:D_SOD-523, symbol Diode:ESD5Zxx
- added IC102: USBLC6-2P6, Package_TO_SOT_SMD:SOT-666, symbol Power_Protection:USBLC6-2P6
- added SB101: Resetn, Jumper:SolderJumper-2_P1.3mm_Open_RoundedPad1.0x1.5mm, symbol Device:R_Small
- added SB102: SWDCLK, Jumper:SolderJumper-2_P1.3mm_Open_RoundedPad1.0x1.5mm, symbol Device:R_Small
- added SB103: SWDIO, Jumper:SolderJumper-2_P1.3mm_Open_RoundedPad1.0x1.5mm, symbol Device:R_Small
- renumbered D107 to D103, D108 to D104, IC102 to IC103, IC103 to IC104, IC104 to IC105, IC105 to IC106, IC106 to IC107, IC107 to IC108, IC108 to IC109
Connections:
- net GND: now also IC102.2 (GND)
- net RESETn: now also SB101.1
- net RESETn_{LV}: now also SB101.2
- net SWDCLK_{LV}: now also SB102.2
- net SWDIO_{LV}: now also SB103.2
- net at C107.1, D101.1 (K), IC105.13 (VCCB)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: now also IC102.5 (VBUS)
- net at X101.2 (SWDIO/TMS): now also IC102.4 (I/O2); no longer IC105.8 (B4)
- net at X101.4 (SWCLK/TCK): now also IC102.6 (I/O1); no longer IC105.10 (B3)
- new net: IC102.1 (I/O1), IC105.10 (B3), SB102.1
- new net: IC102.3 (I/O2), IC105.8 (B4), SB103.1
Other:
- moved on the sheet: C101, C103, C104, C105, C106, IC103, R101, R102, S101, X102

Commit message: Feature: Issue #52
Signed-off-by: Daniel Kampert <DanielKampert@kampis-elektroecke.de>
Parts:
- added R120, R121: 22R, Resistor_SMD:R_0603_1608Metric, symbol Device:R_Small
- SB101, SB102, SB103: symbol Device:R_Small -> Jumper:SolderJumper_2_Open
Connections:
- net RESETn: now also D101.2 (A), D102.1 (K), IC105.11 (B2), X101.10 (~{RESET})
- net at IC102.4 (I/O2): now also R120.1; no longer X101.2 (SWDIO/TMS)
- net at X101.4 (SWCLK/TCK): now also R121.2; no longer IC102.6 (I/O1)
- new net: R120.2, X101.2 (SWDIO/TMS)
- new net: IC102.6 (I/O1), R121.1
Other:
- moved on the sheet: D101, D102, IC102, X101
