File: hardware/Project Architecture.kicad_sch (KiCad schematic)
At the start: 0 parts

Commit message: Issue #51, Clean up Copy+Paste errors in Schematics
Other:
- sheet Main ports: added none; removed BMI270-INT, Buttons, Data, LIS2MDL-INT, MCLK, MIC-CLK, MIC-DATA, MIC-EN, SCL, SDA, VBAT, VIB-EN, VIB-PWM, VSYS, WS, ~{RTC-INT}
Changed lines of the file:
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@@
 	)
 	(arc
-		(start 33.02 33.02)
-		(mid 33.7639 31.2239)
-		(end 35.56 30.48)
+		(start 115.57 74.93)
+		(mid 116.3139 73.1339)
+		(end 118.11 72.39)
 		(stroke
 			(width 0)
@@
 	)
 	(arc
-		(start 35.56 60.96)
-		(mid 33.7698 60.2102)
-		(end 33.02 58.42)
+		(start 118.11 102.87)
+		(mid 116.3198 102.1202)
+		(end 115.57 100.33)
 		(stroke
 			(width 0)
@@
 	)
 	(arc
-		(start 31.75 45.72)
-		(mid 32.6451 46.0949)
-		(end 33.02 46.99)
+		(start 114.3 87.63)
+		(mid 115.1951 88.0049)
+		(end 115.57 88.9)
 		(stroke
 			(width 0)
@@
 	)
 	(arc
-		(start 33.02 44.45)
-		(mid 32.6451 45.3451)
-		(end 31.75 45.72)
+		(start 115.57 86.36)
+		(mid 115.1951 87.2551)
+		(end 114.3 87.63)
 		(stroke
 			(width 0)
@@
 	(text "Page 4"
 		(exclude_from_sim no)
-		(at 57.785 74.93 0)
+		(at 140.335 116.84 0)
 		(effects
 			(font
@@
 		)
 	)
-	(text_box "I2C addresses\n----------------\nBMP581			0x46\nRV-8263-C8		0x51\nAPDS-9306-065	0x52\nBMI270			0x68\nnPM1300			0x6B\nLIS2MDLTR		0x1E"
-		(exclude_from_sim no)
-		(at 247.65 125.73 0)
-		(size 35.56 29.21)
-		(margins 2 2 2 2)
-		(stroke
-			(width 1)
-			(type solid)
-			(color 200 200 200 1)
-		)
-		(fill
-			(type none)
-		)
-		(effects
-			(font
-				(face "Arial")
-				(size 2 2)
-				(color 0 0 0 1)
-			)
-			(justify left top)
-		)
-	)
 	(text_box "Description"
 		(exclude_from_sim no)
-		(at 13.97 43.18 0)
+		(at 96.52 85.09 0)
 		(size 17.145 5.08)
 		(margins 1.4287 1.4287 1.4287 1.4287)
@@
 	(polyline
 		(pts
-			(xy 33.02 46.99) (xy 33.02 58.42)
+			(xy 115.57 88.9) (xy 115.57 100.33)
 		)
 		(stroke
@@
 	(polyline
 		(pts
-			(xy 33.02 44.45) (xy 33.02 33.02)
+			(xy 115.57 86.36) (xy 115.57 74.93)
 		)
 		(stroke
@@
 	)
 	(sheet
-		(at 43.18 17.78)
+		(at 125.73 59.69)
 		(size 38.1 58.42)
 		(exclude_from_sim no)
@@
 		)
 		(property "Sheetname" "Main"
-			(at 43.18 17.0684 0)
+			(at 125.73 58.9784 0)
 			(effects
 				(font
@@
 		)
 		(property "Sheetfile" "Main.kicad_sch"
-			(at 43.18 76.7846 0)
+			(at 125.73 118.6946 0)
 			(effects
 				(font
@@
 			)
 		)
-		(pin "SDA" bidirectional
-			(at 81.28 62.23 0)
-			(effects
-				(font
-					(size 1.27 1.27)
-				)
-				(justify right)
-			)
-		)
-		(pin "SCL" input
-			(at 81.28 59.69 0)
-			(effects
-				(font
-					(size 1.27 1.27)
-				)
-				(justify right)
-			)
-		)
-		(pin "LIS2MDL-INT" output
-			(at 81.28 44.45 0)
-			(effects
-				(font
-					(size 1.27 1.27)
-				)
-				(justify right)
-			)
-		)
-		(pin "BMI270-INT" output
-			(at 81.28 41.91 0)
-			(effects
-				(font
-					(size 1.27 1.27)
-				)
-				(justify right)
-			)
-		)
-		(pin "MIC-EN" input
-			(at 81.28 30.48 0)
-			(effects
-				(font
-					(size 1.27 1.27)
-				)
-				(justify right)
-			)
-		)
-		(pin "MIC-CLK" input
-			(at 81.28 35.56 0)
-			(effects
-				(font
-					(size 1.27 1.27)
-				)
-				(justify right)
-			)
-		)
-		(pin "MIC-DATA" output
-			(at 81.28 33.02 0)
-			(effects
-				(font
-					(size 1.27 1.27)
-				)
-				(justify right)
-			)
-		)
-		(pin "Buttons" output
-			(at 81.28 66.04 0)
-			(effects
-				(font
-					(size 1.27 1.27)
-				)
-				(justify right)
-			)
-		)
-		(pin "VBAT" input
-			(at 81.28 22.86 0)
-			(effects
-				(font
-					(size 1.27 1.27)
-				)
-				(justify right)
-			)
-		)
-		(pin "VSYS" input
-			(at 81.28 25.4 0)
-			(effects
-				(font
-					(size 1.27 1.27)
-				)
-				(justify right)
-			)
-		)
-		(pin "~{RTC-INT}" output
-			(at 81.28 46.99 0)
-			(effects
-				(font
-					(size 1.27 1.27)
-				)
-				(justify right)
-			)
-		)
-		(pin "VIB-EN" input
-			(at 81.28 53.34 0)
-			(effects
-				(font
-					(size 1.27 1.27)
-				)
-				(justify right)
-			)
-		)
-		(pin "VIB-PWM" input
-			(at 81.28 55.88 0)
-			(effects
-				(font
-					(size 1.27 1.27)
-				)
-				(justify right)
-			)
-		)
-		(pin "MCLK" input
-			(at 81.28 69.85 0)
-			(effects
-				(font
-					(size 1.27 1.27)
-				)
-				(justify right)
-			)
-		)
-		(pin "WS" output
-			(at 81.28 72.39 0)
-			(effects
-				(font
-					(size 1.27 1.27)
-				)
-				(justify right)
-			)
-		)
-		(pin "Data" output
-			(at 81.28 74.93 0)
-			(effects
-				(font
-					(size 1.27 1.27)
-				)
-				(justify right)
-			)
-		)
