File: hardware/Main.kicad_sch (KiCad schematic)
At the start: 67 parts, among them IC101 TLV70218_SOT23-5, IC102 USBLC6-2P6, IC103 FT230XQ, IC104 MIC5219-3.3YM5, IC105 NL3V4T244MU2TAG-Q, IC106 USBLC6-2P6, IC107 USB2512BT, IC108 USBLC6-2P6, IC109 MIC2026-1xM, J101 Jumper, J102 Voltage, Q101 BSH205G2AR, SW101 Charge, X101 Debug, X102 UART, X103 Host, X104 Device, X105 Current, Y101 24 MHz

Commit message: Feature: Issue #58
Signed-off-by: Daniel Kampert <DanielKampert@kampis-elektroecke.de>
Parts:
- D103: manf Wurth Elektronik -> ams OSRAM; manf# 150060GS75020 -> LG L29K-G2J1-24; mouser# 710-150060GS75020 -> 720-LGL29KG2J124Z
Changed lines of the file:
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@@
 			)
 		)
-		(property "Datasheet" "https://www.we-online.com/components/products/datasheet/150060GS75020.pdf"
+		(property "Datasheet" "https://www.mouser.de/datasheet/2/588/LG_L29K_EN-3419084.pdf"
 			(at 181.61 200.66 0)
 			(effects
@@
 			)
 		)
-		(property "manf" "Wurth Elektronik"
+		(property "manf" "ams OSRAM"
 			(at 181.61 200.66 0)
 			(effects
@@
 			)
 		)
-		(property "manf#" "150060GS75020"
+		(property "manf#" "LG L29K-G2J1-24"
 			(at 181.61 200.66 0)
 			(effects
@@
 			)
 		)
-		(property "mouser#" "710-150060GS75020"
+		(property "mouser#" "720-LGL29KG2J124Z"
 			(at 181.61 200.66 0)
 			(effects

Commit message: Issue #51, Clean up Copy+Paste errors in Schematics
Connections:
- net V_{Watch}: now also IC108.5 (VBUS)
- net at Q101.1 (G), R117.1, SW101.3 (C): now also D104.1 (K)
- net at R115.2, X104.A4 (VBUS), X104.A9 (VBUS)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: no longer IC108.5 (VBUS)
- net at SW101.1 (A): no longer D104.1 (K)
- no-connect marks 22 -> 23
Changed lines of the file:
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@@
 	)
 	(junction
+		(at 339.09 50.8)
+		(diameter 0)
+		(color 0 0 0 0)
+	)
+	(junction
 		(at 119.38 87.63)
 		(diameter 0)
@@
 	)
 	(junction
-		(at 295.91 29.21)
-		(diameter 0)
-		(color 0 0 0 0)
-	)
-	(junction
 		(at 252.73 54.61)
 		(diameter 0)
@@
 	)
 	(no_connect
+		(at 344.17 54.61)
+	)
+	(no_connect
 		(at 166.37 77.47)
 	)
@@
 	(wire
 		(pts
+			(xy 295.91 38.1) (xy 297.18 38.1)
+		)
+		(stroke
+			(width 0)
+			(type default)
+		)
+	)
+	(wire
+		(pts
 			(xy 125.73 68.58) (xy 125.73 69.85)
 		)
@@
 	(wire
 		(pts
-			(xy 339.09 39.37) (xy 339.09 54.61)
+			(xy 339.09 39.37) (xy 339.09 50.8)
 		)
 		(stroke
@@
 	(wire
 		(pts
-			(xy 344.17 54.61) (xy 344.17 50.8)
-		)
-		(stroke
-			(width 0)
-			(type default)
-		)
-	)
-	(wire
-		(pts
 			(xy 363.22 172.72) (xy 363.22 175.26)
 		)
@@
 	(wire
 		(pts
-			(xy 344.17 50.8) (xy 345.44 50.8)
-		)
-		(stroke
-			(width 0)
-			(type default)
-		)
-	)
-	(wire
-		(pts
 			(xy 331.47 203.2) (xy 331.47 208.28)
 		)
@@
 	(wire
 		(pts
-			(xy 250.19 29.21) (xy 295.91 29.21)
-		)
-		(stroke
-			(width 0)
-			(type default)
-		)
-	)
-	(wire
-		(pts
 			(xy 181.61 204.47) (xy 181.61 208.28)
 		)
@@
 	(wire
 		(pts
+			(xy 295.91 38.1) (xy 295.91 39.37)
+		)
+		(stroke
+			(width 0)
+			(type default)
+		)
+	)
+	(wire
+		(pts
 			(xy 339.09 36.83) (xy 339.09 39.37)
 		)
@@
 	(wire
 		(pts
-			(xy 295.91 29.21) (xy 321.31 29.21)
+			(xy 250.19 29.21) (xy 321.31 29.21)
 		)
 		(stroke
@@
 	(wire
 		(pts
+			(xy 339.09 50.8) (xy 345.44 50.8)
+		)
+		(stroke
+			(width 0)
+			(type default)
+		)
+	)
+	(wire
+		(pts
 			(xy 30.48 69.85) (xy 63.5 69.85)
 		)
@@
 	(wire
 		(pts
-			(xy 295.91 29.21) (xy 295.91 39.37)
-		)
-		(stroke
-			(width 0)
-			(type default)
-		)
-	)
-	(wire
-		(pts
 			(xy 29.21 72.39) (xy 40.64 72.39)
 		)
@@
 	(wire
 		(pts
+			(xy 339.09 50.8) (xy 339.09 54.61)
+		)
+		(stroke
+			(width 0)
+			(type default)
+		)
+	)
+	(wire
+		(pts
 			(xy 251.46 43.18) (xy 287.02 43.18)
 		)
@@
 		)
 	)
+	(global_label "V_{Watch}"
+		(shape input)
+		(at 297.18 38.1 0)
+		(fields_autoplaced yes)
+		(effects
+			(font
+				(size 1.27 1.27)
+			)
+			(justify left)
+		)
+		(property "Intersheetrefs" "${INTERSHEET_REFS}"
+			(at 305.1014 38.1 0)
+			(effects
+				(font
+					(size 1.27 1.27)
+				)
+				(justify left)
+				(hide yes)
+			)
+		)
+	)
 	(symbol
 		(lib_id "power:+3V3")
@@
 			)
 		)
-		(property "Description" ""
+		(property "Description" "-2A Id, -20V Vds, P-Channel MOSFET, SOT-23"
 			(at 339.09 29.21 0)
 			(effects
@@
 			(at 339.09 29.21 0)
 			(effects
+				(font
+					(size 1.27 1.27)
+				)
+				(hide yes)
+			)
+		)
+		(property "CONFIG" ""
+			(at 339.09 29.21 0)
+			(effects

Commit message: Feature: Issue #59
Signed-off-by: Daniel Kampert <DanielKampert@kampis-elektroecke.de>
Parts:
- removed IC105: NL3V4T244MU2TAG-Q, Package_SO:TSSOP-14_4.4x5mm_P0.65mm, symbol ON Semiconductor:NL3V4T244 (TSSOP14)
- added IC405: TXB0304RUT, Package_DFN_QFN:Texas_R-PUQFN-N12, symbol Logic_LevelTranslator:TXB0304RUT
- R405: renamed from R103; now fitted
- R406: renamed from R104; now not fitted; now left out of the parts list
- renumbered C101 to C401, C102 to C402, C103 to C403, C104 to C404, C105 to C405, C107 to C406, C106 to C407, C108 to C408, C109 to C409, C110 to C410, C111 to C411, C112 to C412, C113 to C413, C114 to C414, C115 to C415, C116 to C416, C117 to C417, C118 to C418, C119 to C419, D101 to D401, D102 to D402, D103 to D403, D104 to D404, IC101 to IC401, IC102 to IC402, IC103 to IC403, IC104 to IC404, IC106 to IC406, IC107 to IC407, IC108 to IC408, IC109 to IC409, J101 to J401, J102 to J402, Q101 to Q401, R101 to R401, R121 to R402, R120 to R403, R102 to R404, R107 to R407, R108 to R408, R105 to R409, R106 to R410, R109 to R411, R110 to R412, R111 to R413, R112 to R414, R113 to R415, R114 to R416, R116 to R417, R115 to R418, R119 to R419, R117 to R420, R118 to R421, S101 to S401, SB101 to SB401, SB102 to SB402, SB103 to SB403, SW101 to SW401, X101 to X401, X102 to X402, X103 to X403, X104 to X404, X105 to X405, Y101 to Y401
Connections:
- net +1V8: now also IC405.1 (VCCA)
- net GND: now also IC405.6 (GND)
- net RESETn: now also IC405.10 (B1), IC405.9 (B2)
- net RESETn_{LV}: now also IC405.2 (A1), IC405.3 (A2)
- net SWDCLK_{LV}: now also IC405.4 (A3)
- net SWDIO_{LV}: now also IC405.5 (A4)
- net at C406.1, D401.1 (K), IC402.5 (VBUS)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: now also IC405.11 (VCCB)
- net at IC402.1 (I/O1), SB402.1 (A): now also IC405.8 (B3)
- net at R405.2, R406.1: now also IC405.12 (OE)
- net at IC402.3 (I/O2), SB403.1 (A): now also IC405.7 (B4)
Other:
- note added: "Swap these resistors when using the TXBN variant!"
- moved on the sheet: C406, D404, IC406, IC408, Q401, R409, R410, R415, R416, R418, R420, R421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

Commit message: Issue #61
Parts:
- X404: footprint Connector_USB:USB_C_Receptacle_Amphenol_12401610E4-2A -> Amphenol:10133475-10001LF; manf# 12401610E4-2A -> 10133475-10001LF; mouser# 523-12401610E4#2A -> 523-10133475-10001LF
Changed lines of the file:
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@@
 			)
 		)
-		(property "Footprint" "Connector_USB:USB_C_Receptacle_Amphenol_12401610E4-2A"
+		(property "Footprint" "Amphenol:10133475-10001LF"
 			(at 267.97 54.61 0)
 			(effects
@@
 			)
 		)
-		(property "Datasheet" "https://www.usb.org/sites/default/files/documents/usb_type-c.zip"
+		(property "Datasheet" "https://cdn.amphenol-cs.com/media/wysiwyg/files/drawing/10133475.pdf"
 			(at 267.97 54.61 0)
 			(effects
@@
 			)
 		)
-		(property "Description" "USB Full-Featured Type-C Receptacle connector"
+		(property "Description" "USB Full-Featured Type-C edge connector"
 			(at 264.16 54.61 0)
 			(effects
@@
 			)
 		)
-		(property "manf#" "12401610E4-2A"
+		(property "manf#" "10133475-10001LF"
 			(at 264.16 54.61 0)
 			(effects
@@
 			)
 		)
-		(property "mouser#" "523-12401610E4#2A"
+		(property "mouser#" "523-10133475-10001LF"
 			(at 264.16 54.61 0)
 			(effects
