File: dock/Main.kicad_sch (KiCad schematic)
At the start: 67 parts, among them IC401 TLV70218_SOT23-5, IC402 USBLC6-2P6, IC403 FT230XQ, IC404 MIC5219-3.3YM5, IC405 TXB0304RUT, IC406 USBLC6-2P6, IC407 USB2512BT, IC408 USBLC6-2P6, IC409 MIC2026-1xM, J401 Jumper, J402 Voltage, Q401 BSH205G2AR, SW401 Charge, X401 Debug, X402 UART, X403 Host, X404 Device, X405 Current, Y401 24 MHz

Commit message: Working on CI/CD pipeline
Parts:
- IC407: manf# USB2512BT/M2 -> USB2512BT/M2
- J401: manf Würth Elektronik -> Würth Elektronik
- R418: manf Vishay -> Bourns; manf# CRCW08050000Z0EAHP -> CR0805-J/-000ELF; mouser# 71-CRCW08050000Z0EAHP -> 652-CR0805-J/-000ELF
Other:
- note removed: "Configuration: - All ports are non-removable (REM0 = low and REM1 = high) - LED is active low (REM0 = low and REM1 = high) - Strap options enabled (CFG_SEL0 and CFG_SEL1 = low) - Self-powered operation enabled (CFG_SEL0 and CFG_SEL1 = low) - Individual power switching enabled (CFG_SEL0 and CFG_SEL1 = low) - Individual over-current sensing enabled (CFG_SEL0 and CFG_SEL1 = low) - Enable battery opt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"
- moved on the sheet: C412, C413, C414, C415, C416, C417, C418, C419, D403, IC407, IC409, R407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
