File: dock/Main.kicad_sch (KiCad schematic)
At the start: 67 parts, among them IC401 TLV70218_SOT23-5, IC402 USBLC6-2P6, IC403 FT230XQ, IC404 MIC5219-3.3YM5, IC405 TXB0304RUT, IC406 USBLC6-2P6, IC407 USB2512BT, IC408 USBLC6-2P6, IC409 MIC2026-1xM, J401 Jumper, J402 Voltage, Q401 BSH205G2AR, SW401 Charge, X401 Debug, X402 UART, X403 Host, X404 Device, X405 Current, Y401 24 MHz

Commit message: Bug: Issue #48
- Flip Rx and Tx lines for UART and SWD
- Update .gitignore

Closes #48

Signed-off-by: Daniel Kampert <DanielKampert@kampis-elektroecke.de>
Connections:
- net RxD_{LV}: now also X404.A2 (TX1+), X404.B2 (TX2+); no longer X404.A11 (RX2+), X404.B11 (RX1+)
- net SWDCLK_{LV}: now also X404.A11 (RX2+), X404.B11 (RX1+); no longer X404.A2 (TX1+), X404.B2 (TX2+)
- net SWDIO_{LV}: now also X404.A10 (RX2-), X404.B10 (RX1-); no longer X404.A3 (TX1-), X404.B3 (TX2-)
- net TxD_{LV}: now also X404.A3 (TX1-), X404.B3 (TX2-); no longer X404.A10 (RX2-), X404.B10 (RX1-)
Changed lines of the file:
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@@
 	(global_label "TxD_{LV}"
 		(shape input)
-		(at 285.75 54.61 0)
-		(fields_autoplaced yes)
-		(effects
-			(font
-				(size 1.27 1.27)
-			)
-			(justify left)
-		)
-		(property "Intersheetrefs" "${INTERSHEET_REFS}"
-			(at 293.0909 54.61 0)
+		(at 285.75 77.47 0)
+		(fields_autoplaced yes)
+		(effects
+			(font
+				(size 1.27 1.27)
+			)
+			(justify left)
+		)
+		(property "Intersheetrefs" "${INTERSHEET_REFS}"
+			(at 293.0909 77.47 0)
 			(effects
 				(font
@@
 	(global_label "SWDCLK_{LV}"
 		(shape input)
-		(at 285.75 64.77 0)
-		(fields_autoplaced yes)
-		(effects
-			(font
-				(size 1.27 1.27)
-			)
-			(justify left)
-		)
-		(property "Intersheetrefs" "${INTERSHEET_REFS}"
-			(at 297.3242 64.77 0)
+		(at 285.75 57.15 0)
+		(fields_autoplaced yes)
+		(effects
+			(font
+				(size 1.27 1.27)
+			)
+			(justify left)
+		)
+		(property "Intersheetrefs" "${INTERSHEET_REFS}"
+			(at 297.3242 57.15 0)
 			(effects
 				(font
@@
 	(global_label "RxD_{LV}"
 		(shape output)
-		(at 285.75 57.15 0)
-		(fields_autoplaced yes)
-		(effects
-			(font
-				(size 1.27 1.27)
-			)
-			(justify left)
-		)
-		(property "Intersheetrefs" "${INTERSHEET_REFS}"
-			(at 293.3933 57.15 0)
+		(at 285.75 64.77 0)
+		(fields_autoplaced yes)
+		(effects
+			(font
+				(size 1.27 1.27)
+			)
+			(justify left)
+		)
+		(property "Intersheetrefs" "${INTERSHEET_REFS}"
+			(at 293.3933 64.77 0)
 			(effects
 				(font
@@
 	(global_label "SWDIO_{LV}"
 		(shape bidirectional)
-		(at 285.75 77.47 0)
-		(fields_autoplaced yes)
-		(effects
-			(font
-				(size 1.27 1.27)
-			)
-			(justify left)
-		)
-		(property "Intersheetrefs" "${INTERSHEET_REFS}"
-			(at 296.6439 77.47 0)
-			(effects
-				(font
+		(at 285.75 54.61 0)
+		(fields_autoplaced yes)
+		(effects
+			(font
+				(size 1.27 1.27)
+			)
+			(justify left)
+		)
+		(property "Intersheetrefs" "${INTERSHEET_REFS}"
+			(at 296.6439 54.61 0)
+			(effects
+				(font

Commit message: Task: Issue #69
- Change ZSWatch USB to a single sided and more stable one

Closes #69

Signed-off-by: Daniel Kampert <DanielKampert@kampis-elektroecke.de>
Parts:
- removed R415, R416: 5k1, Resistor_SMD:R_0603_1608Metric, symbol Device:R_Small
- X404: footprint Amphenol:10133475-10001LF -> GlobTect:PLUG-USBC-241SMT-4BC2SS; digikey# (none) -> 1939-PLUG-USBC-241SMT-4BC2SSCT-ND; manf Amphenol Commercial Products -> GlobTek, Inc.; manf# 10133475-10001LF -> PLUG-USBC-241SMT-4BC2SS; mouser# 523-10133475-10001LF -> (none)
Connections:
- net D_{2}+: no longer X404.B6 (D+)
- net D_{2}-: no longer X404.B7 (D-)
- net RESETn_{LV}: no longer X404.B8 (SBU2)
- net RxD_{LV}: no longer X404.B2 (TX2+)
- net SWDCLK_{LV}: no longer X404.B11 (RX1+)
- net SWDIO_{LV}: no longer X404.B10 (RX1-)
- net TxD_{LV}: no longer X404.B3 (TX2-)
- no-connect marks 23 -> 32
Other:
- moved on the sheet: IC408
