File: dock/ZSWatch-Dock.kicad_pcb (KiCad board)
At the start: 4 copper layers, 80 x 48 mm, 75 parts, among them IC401 TLV70218_SOT23-5, IC402 USBLC6-2P6, IC403 FT230XQ, IC404 MIC5219-3.3YM5, IC405 TXB0304RUT, IC406 USBLC6-2P6, IC407 USB2512BT, IC408 USBLC6-2P6, IC409 MIC2026-1xM, J402 Voltage, Q401 BSH205G2AR, SW401 Charge, X401 Debug, X402 UART, X403 Host, X404 Device, X405 Current, Y401 24 MHz

Commit message: Update outputs (release)
Other:
- board text added: "0.1855mm"
- board text added: "0.23mm"
- board text added: "Inner1"
- board text added: "Inner2"
- board text added: "Plane"
- board text added: "Prepreg"
- board text added: "Total thickness: 0.761mm"
- board text removed: "1.51mm"
- board text removed: "Total thickness: 1.6mm"

Commit message: Bug: Issue #48
- Flip Rx and Tx lines for UART and SWD
- Update .gitignore

Closes #48

Signed-off-by: Daniel Kampert <DanielKampert@kampis-elektroecke.de>
Connections:
- X404 pad A10: TxD_{LV} -> SWDIO_{LV}
- X404 pad A11: RxD_{LV} -> SWDCLK_{LV}
- X404 pad A2: SWDCLK_{LV} -> RxD_{LV}
- X404 pad A3: SWDIO_{LV} -> TxD_{LV}
- X404 pad B10: TxD_{LV} -> SWDIO_{LV}
- X404 pad B11: RxD_{LV} -> SWDCLK_{LV}
- X404 pad B2: SWDCLK_{LV} -> RxD_{LV}
- X404 pad B3: SWDIO_{LV} -> TxD_{LV}
Routing:
- net RxD_{LV}: track 95.5 -> 85.2 mm, vias 5 -> 4
- net TxD_{LV}: track 75.8 -> 70.2 mm
- net Net-(X404-CC2): track 10.6 -> 7.94 mm
- net GND: track 59.1 -> 59.6 mm
Other:
- board text added: "1.51mm"
- board text added: "Total thickness: 1.6mm"
- board text removed: "0.1855mm"
- board text removed: "0.23mm"
- board text removed: "Inner1"
- board text removed: "Inner2"
- board text removed: "Plane"
- board text removed: "Prepreg"
- board text removed: "Total thickness: 0.761mm"

Commit message: Task: Issue #69
- Change ZSWatch USB to a single sided and more stable one

Closes #69

Signed-off-by: Daniel Kampert <DanielKampert@kampis-elektroecke.de>
Parts:
- removed R415, R416: 5k1, Resistor_SMD:R_0603_1608Metric
- X404: footprint Amphenol:10133475-10001LF -> GlobTect:PLUG-USBC-241SMT-4BC2SS
- moved X404 1.49 mm to (167.8, 147.1)
- moved IC408 1.29 mm to (177.1, 147.1)
Connections:
- X404 pad A5: Net-(X404-CC1) -> unconnected-(X404-CC1-PadA5)
- X404 pad B10: SWDIO_{LV} -> unconnected-(X404-RX1--PadB10)
- X404 pad B11: SWDCLK_{LV} -> unconnected-(X404-RX1+-PadB11)
- X404 pad B2: RxD_{LV} -> unconnected-(X404-TX2+-PadB2)
- X404 pad B3: TxD_{LV} -> unconnected-(X404-TX2--PadB3)
- X404 pad B5: Net-(X404-CC2) -> unconnected-(X404-CC2-PadB5)
- X404 pad B6: /Project Architecture/Main/D_{2}+ -> unconnected-(X404-D+-PadB6)
- X404 pad B7: /Project Architecture/Main/D_{2}- -> unconnected-(X404-D--PadB7)
- X404 pad B8: RESETn_{LV} -> unconnected-(X404-SBU2-PadB8)
Routing:
- net RxD_{LV}: track 85.2 -> 68.3 mm
- net TxD_{LV}: track 70.2 -> 54.6 mm
- net RESETn_{LV}: track 51.7 -> 39.7 mm, vias 5 -> 2
- net SWDIO_{LV}: track 47.5 -> 36.5 mm, vias 3 -> 2
- net SWDCLK_{LV}: track 44.2 -> 34.4 mm, vias 4 -> 3
- net /Project Architecture/Main/D_{2}+: track 14.6 -> 6.28 mm
- net Net-(X404-CC1): track 7.97 -> 0.00 mm
- net Net-(X404-CC2): track 7.94 -> 0.00 mm, vias 1 -> 0
- net /Project Architecture/Main/D_{2}-: track 13.6 -> 6.24 mm, vias 1 -> 0
- net Net-(X405-Pin_1): track 34.3 -> 28.2 mm, vias 3 -> 0
- net V_{Watch}: track 166.5 -> 160.9 mm
- net GND: track 59.6 -> 60.7 mm, vias 45 -> 43
- net USB-2-D-: track 50.1 -> 49.5 mm
- net USB-2-D+: track 50.8 -> 50.1 mm
Other:
- outline, holes or cut-outs redrawn

Commit message: Task: Issue #72
- Move Voltage REF connector a little

Closes #72

Signed-off-by: Daniel Kampert <DanielKampert@kampis-elektroecke.de>
Parts:
- moved J402 2.60 mm to (216.1, 125.9)
Routing:
- net Net-(D401-K): track 29.6 -> 32.2 mm
- net +1V8: track 74.9 -> 74.0 mm
Changed lines of the file:
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@@
 	(footprint "Connector_PinHeader_2.54mm:PinHeader_1x03_P2.54mm_Vertical"
 		(layer "F.Cu")
-		(at 213.5 125.9)
+		(at 216.1 125.9)
 		(descr "Through hole straight pin header, 1x03, 2.54mm pitch, single row")
 		(tags "Through hole pin header THT 1x03 2.54mm single row")
@@
 	)
 	(gr_text "+3V3"
-		(at 215.2 125.9 0)
+		(at 217.8 125.9 0)
 		(layer "F.SilkS")
 		(effects
@@
 	)
 	(gr_text "+1V8"
-		(at 215.2 130.98 0)
+		(at 217.8 130.98 0)
 		(layer "F.SilkS")
 		(effects
@@
 	)
 	(segment
-		(start 189.65 138.1)
-		(end 189.65 130.3)
-		(width 0.2)
-		(layer "F.Cu")
-		(net 2)
-	)
-	(segment
 		(start 190.995 127.2)
 		(end 191.6375 127.8425)
@@
 	)
 	(segment
-		(start 219.2125 136.675)
-		(end 218.225 136.675)
+		(start 216.1 136.7)
+		(end 216.1 130.98)
 		(width 0.2)
 		(layer "F.Cu")
@@
 	)
 	(segment
-		(start 203.9 152.025)
-		(end 208.95 152.025)
+		(start 216.125 136.725)
+		(end 217.45 136.725)
 		(width 0.2)
 		(layer "F.Cu")
@@
 	)
 	(segment
-		(start 208.95 152.025)
-		(end 208.975 152)
+		(start 216.1 136.7)
+		(end 216.125 136.725)
+		(width 0.2)
+		(layer "F.Cu")
+		(net 2)
+	)
+	(segment
+		(start 219.2125 136.675)
+		(end 218.225 136.675)
 		(width 0.2)
 		(layer "F.Cu")
@@
 	)
 	(segment
-		(start 213.5 130.98)
-		(end 213.5 138.1)
+		(start 203.9 152.025)
+		(end 208.95 152.025)
 		(width 0.2)
 		(layer "F.Cu")
@@
 	)
 	(segment
-		(start 216.075 138.1)
-		(end 217.45 136.725)
+		(start 208.95 152.025)
+		(end 208.975 152)
 		(width 0.2)
 		(layer "F.Cu")
@@
 	)
 	(segment
-		(start 213.5 138.1)
-		(end 216.075 138.1)
+		(start 190.2 125.2)
+		(end 190.2 126.1)
 		(width 0.2)
 		(layer "F.Cu")
@@
 	)
 	(segment
-		(start 190.2 125.2)
-		(end 190.2 126.1)
+		(start 190.4 127.2)
+		(end 189.65 127.2)
 		(width 0.2)
 		(layer "F.Cu")
@@
 	)
 	(segment
-		(start 190.4 127.2)
-		(end 189.65 127.2)
+		(start 189.65 136.7)
+		(end 189.65 130.3)
 		(width 0.2)
 		(layer "F.Cu")
@@
 	)
 	(via
-		(at 189.65 138.1)
+		(at 189.65 136.7)
 		(size 0.45)
 		(drill 0.25)
@@
 	)
 	(via
-		(at 213.5 138.1)
+		(at 216.1 136.7)
 		(size 0.45)
 		(drill 0.25)
@@
 	)
 	(segment
-		(start 213.5 138.1)
-		(end 208.975 142.625)
+		(start 189.65 136.7)
+		(end 216.1 136.7)
 		(width 0.2)
 		(layer "B.Cu")
@@
 	)
 	(segment
-		(start 208.975 142.625)
+		(start 208.975 145.225)
 		(end 208.975 152.025)
 		(width 0.2)
@@
 	)
 	(segment
-		(start 189.65 138.1)
-		(end 213.5 138.1)
+		(start 216.1 136.7)
+		(end 216.1 138.1)
+		(width 0.2)
+		(layer "B.Cu")
+		(net 2)
+	)
+	(segment
+		(start 216.1 138.1)
+		(end 208.975 145.225)
 		(width 0.2)
 		(layer "B.Cu")
@@
 	)
 	(segment
+		(start 210.18 126.5)
+		(end 214.16 126.5)
+		(width 0.2)
+		(layer "F.Cu")
+		(net 20)
+	)
+	(segment
 		(start 199.0625 130.6625)
 		(end 199.325 130.6625)
@@
 	)
 	(segment
-		(start 210.18 126.5)
-		(end 211.56 126.5)
-		(width 0.2)
-		(layer "F.Cu")
-		(net 20)
-	)
-	(segment
 		(start 201.7 124.7)
 		(end 209.9 124.7)
@@
 	)
 	(segment
-		(start 211.56 126.5)
-		(end 213.5 128.44)
+		(start 195.1 126.3)
+		(end 194.2 127.2)
 		(width 0.2)
 		(layer "F.Cu")
@@
 	)
 	(segment
-		(start 195.1 126.3)
-		(end 194.2 127.2)
+		(start 210.18 124.98)
+		(end 210.18 126.5)
 		(width 0.2)
 		(layer "F.Cu")
@@
 	)
 	(segment
-		(start 210.18 124.98)
-		(end 210.18 126.5)
+		(start 214.16 126.5)
+		(end 216.1 128.44)
 		(width 0.2)
 		(layer "F.Cu")
